File: Electrical/Electrical.kicad_pcb (KiCad board)
At the start: 2 copper layers, 26 x 30 mm, 11 parts, among them P1 USB_C_Plug_USB2.0, U1 AP2112K-3.3

Commit message: update Setup
Parts:
- added REF**: ublox_MAX, RF_GPS:ublox_MAX, F.Cu at (139.7, 149.9)
- added REF**: QFN-56-1EP_7x7mm_P0.4mm_EP3.2x3.2mm, Package_DFN_QFN:QFN-56-1EP_7x7mm_P0.4mm_EP3.2x3.2mm, F.Cu at (147.3, 137.2)
