File: Electrical/_autosave-Electrical.kicad_sch (KiCad schematic)
At the start: 13 parts, among them P1 USB_C_Plug_USB2.0, U1 AP2112K-3.3

Commit message: updated Setup.md
Parts:
- removed U?: TUSB2036, Package_QFP:LQFP-32_7x7mm_P0.8mm, symbol Interface_USB:TUSB2036
- added J?: USB_C_Receptacle_USB2.0, symbol Connector:USB_C_Receptacle_USB2.0
- added U?: RAK4200, RF_Module:RAK4200, symbol RF_Module:RAK4200
- added U?: L70-R, RF_GPS:Quectel_L70-R, symbol RF_GPS:L70-R
- added U?: TUSB4041I, Package_QFP:HTQFP-64-1EP_10x10mm_P0.5mm_EP8x8mm_Mask4.4x4.4mm_ThermalVias, symbol Interface_USB:TUSB4041I
Connections:
- new net: J?.A1 (GND), J?.A12 (GND), J?.B1 (GND), J?.B12 (GND)
- new net: J?.A4 (VBUS), J?.A9 (VBUS), J?.B4 (VBUS), J?.B9 (VBUS)
- new net: U?.11 (GND), U?.13 (GND), U?.14 (GND), U?.19 (GND)
- new net: U?.1 (GND), U?.10 (GND), U?.12 (GND)
Changed lines of the file:
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@@
     (pin "1")
   )
-  (symbol (lib_id "Interface_USB:TUSB2036") (at 181.61 73.66 0) (unit 1)
-    (in_bom yes) (on_board yes) (fields_autoplaced)
-    (property "Reference" "U?" (id 0) (at 186.1694 33.02 0)
-      (effects (font (size 1.27 1.27)) (justify left))
-    )
-    (property "Value" "TUSB2036" (id 1) (at 186.1694 35.56 0)
-      (effects (font (size 1.27 1.27)) (justify left))
-    )
-    (property "Footprint" "Package_QFP:LQFP-32_7x7mm_P0.8mm" (id 2) (at 208.28 111.76 0)
-      (effects (font (size 1.27 1.27)) hide)
-    )
-    (property "Datasheet" "http://www.ti.com/lit/ds/symlink/tusb2036.pdf" (id 3) (at 181.61 73.66 0)
+  (symbol (lib_id "Connector:USB_C_Receptacle_USB2.0") (at 151.13 151.13 0) (unit 1)
+    (in_bom yes) (on_board yes) (fields_autoplaced)
+    (property "Reference" "J?" (id 0) (at 151.13 128.27 0))
+    (property "Value" "USB_C_Receptacle_USB2.0" (id 1) (at 151.13 130.81 0))
+    (property "Footprint" "" (id 2) (at 154.94 151.13 0)
+      (effects (font (size 1.27 1.27)) hide)
+    )
+    (property "Datasheet" "https://www.usb.org/sites/default/files/documents/usb_type-c.zip" (id 3) (at 154.94 151.13 0)
+      (effects (font (size 1.27 1.27)) hide)
+    )
+    (pin "A1")
+    (pin "A12")
+    (pin "A4")
+    (pin "A5")
+    (pin "A6")
+    (pin "A7")
+    (pin "A8")
+    (pin "A9")
+    (pin "B1")
+    (pin "B12")
+    (pin "B4")
+    (pin "B5")
+    (pin "B6")
+    (pin "B7")
+    (pin "B8")
+    (pin "B9")
+    (pin "S1")
+  )
+  (symbol (lib_id "RF_Module:RAK4200") (at 215.9 135.89 0) (unit 1)
+    (in_bom yes) (on_board yes) (fields_autoplaced)
+    (property "Reference" "U?" (id 0) (at 217.9194 110.49 0)
+      (effects (font (size 1.27 1.27)) (justify left))
+    )
+    (property "Value" "RAK4200" (id 1) (at 217.9194 113.03 0)
+      (effects (font (size 1.27 1.27)) (justify left))
+    )
+    (property "Footprint" "RF_Module:RAK4200" (id 2) (at 220.98 128.27 0)
+      (effects (font (size 1.27 1.27)) hide)
+    )
+    (property "Datasheet" "https://downloads.rakwireless.com/LoRa/RAK4200/Hardware-Specification/RAK4200_Module_Specifications_V1.4.pdf" (id 3) (at 220.98 128.27 0)
+      (effects (font (size 1.27 1.27)) hide)
+    )
+    (pin "1")
+    (pin "10")
+    (pin "11")
+    (pin "12")
+    (pin "13")
+    (pin "14")
+    (pin "15")
+    (pin "16")
+    (pin "17")
+    (pin "18")
+    (pin "19")
+    (pin "2")
+    (pin "20")
+    (pin "3")
+    (pin "4")
+    (pin "5")
+    (pin "6")
+    (pin "7")
+    (pin "8")
+    (pin "9")
+  )
+  (symbol (lib_id "RF_GPS:L70-R") (at 255.27 90.17 0) (unit 1)
+    (in_bom yes) (on_board yes) (fields_autoplaced)
+    (property "Reference" "U?" (id 0) (at 257.2894 105.41 0)
+      (effects (font (size 1.27 1.27)) (justify left))
+    )
+    (property "Value" "L70-R" (id 1) (at 257.2894 107.95 0)
+      (effects (font (size 1.27 1.27)) (justify left))
+    )
+    (property "Footprint" "RF_GPS:Quectel_L70-R" (id 2) (at 255.27 116.84 0)
+      (effects (font (size 1.27 1.27)) hide)
+    )
+    (property "Datasheet" "https://www.quectel.com/product/gps-only-l70-r" (id 3) (at 255.27 120.65 0)
+      (effects (font (size 1.27 1.27)) hide)
+    )
+    (pin "1")
+    (pin "10")
+    (pin "11")
+    (pin "12")
+    (pin "13")
+    (pin "14")
+    (pin "15")
+    (pin "16")
+    (pin "17")
+    (pin "18")
+    (pin "2")
+    (pin "3")
+    (pin "4")
+    (pin "5")
+    (pin "6")
+    (pin "7")
+    (pin "8")
+    (pin "9")
+  )
+  (symbol (lib_id "Interface_USB:TUSB4041I") (at 167.64 71.12 0) (unit 1)
+    (in_bom yes) (on_board yes) (fields_autoplaced)
+    (property "Reference" "U?" (id 0) (at 169.6594 121.92 0)
+      (effects (font (size 1.27 1.27)) (justify left))
+    )
+    (property "Value" "TUSB4041I" (id 1) (at 169.6594 124.46 0)
+      (effects (font (size 1.27 1.27)) (justify left))
+    )
+    (property "Footprint" "Package_QFP:HTQFP-64-1EP_10x10mm_P0.5mm_EP8x8mm_Mask4.4x4.4mm_ThermalVias" (id 2) (at 198.12 20.32 0)
+      (effects (font (size 1.27 1.27)) (justify left) hide)
+    )
+    (property "Datasheet" "http://www.ti.com/lit/ds/symlink/tusb4041i.pdf" (id 3) (at 160.02 66.04 0)
       (effects (font (size 1.27 1.27)) hide)
     )
@@
     (pin "31")
     (pin "32")
+    (pin "33")
+    (pin "34")
+    (pin "35")
+    (pin "36")
+    (pin "37")
+    (pin "38")
+    (pin "39")
     (pin "4")
+    (pin "40")
+    (pin "41")
+    (pin "42")
+    (pin "43")
+    (pin "44")
+    (pin "45")
+    (pin "46")
+    (pin "47")
+    (pin "48")
+    (pin "49")
     (pin "5")
+    (pin "50")
+    (pin "51")
+    (pin "52")
+    (pin "53")
+    (pin "54")
+    (pin "55")
+    (pin "56")
+    (pin "57")
+    (pin "58")
+    (pin "59")
     (pin "6")
+    (pin "60")
+    (pin "61")
+    (pin "62")
+    (pin "63")
+    (pin "64")
+    (pin "65")
     (pin "7")
     (pin "8")
@@
       (reference "H2") (unit 1) (value "MountingHole") (footprint "MountingHole:MountingHole_2.2mm_M2")
     )
+    (path "/3005da1c-9639-4919-a041-792971fb122a"
+      (reference "J?") (unit 1) (value "USB_C_Receptacle_USB2.0") (footprint "")
+    )
     (path "/00000000-0000-0000-0000-00005fd76bc6"
       (reference "P1") (unit 1) (value "USB_C_Plug_USB2.0") (footprint "Expansion_Card:USB_C_Plug_Molex_105444")
@@
       (reference "U1") (unit 1) (value "AP2112K-3.3") (footprint "Package_TO_SOT_SMD:SOT-23-5")
     )
-    (path "/7a04c364-40cd-46c0-b2d4-43b1a14d5b57"
-      (reference "U?") (unit 1) (value "TUSB2036") (footprint "Package_QFP:LQFP-32_7x7mm_P0.8mm")
+    (path "/71cf81b1-28fb-41a9-97fb-4afd92e2de8e"
+      (reference "U?") (unit 1) (value "RAK4200") (footprint "RF_Module:RAK4200")
+    )
+    (path "/7595683d-1201-4c94-aaf5-e2eeaf5eadb3"
+      (reference "U?") (unit 1) (value "L70-R") (footprint "RF_GPS:Quectel_L70-R")
+    )
+    (path "/d8b05be9-691c-48ce-ad74-a5481d3bf5f9"
+      (reference "U?") (unit 1) (value "TUSB4041I") (footprint "Package_QFP:HTQFP-64-1EP_10x10mm_P0.5mm_EP8x8mm_Mask4.4x4.4mm_ThermalVias")
     )
     (path "/ea7d0817-655a-431b-a98b-70b84598125f"
